File: pcb/left.kicad_sch (KiCad schematic)
At the start: 75 parts, among them K1 KEY_ESC, K10 KEY_Z, K11 KEY_LSUP, K12 KEY_W, K13 KEY_S, K14 KEY_X, K15 KEY_LALT, K16 KEY_3, K17 KEY_E, K18 KEY_D, K19 KEY_C, K2 KEY_1, K20 KEY_TL1, K21 KEY_4, K22 KEY_R, K23 KEY_F, K24 KEY_V, K25 KEY_TL2, K26 KEY_5, K27 KEY_T, K28 KEY_G, K29 KEY_B, K3 KEY_2, K30 KEY_TL3, K31 KEY_6, K32 KEY_CL1, K33 KEY_CL2, K34 KEY_CL3, K4 KEY_TAB, K5 KEY_CAPS, K6 KEY_LSFT, K7 KEY_LCTL, K8 KEY_Q, K9 KEY_A, T1 T_MODE, T2 T_SPACE, U1 TRRS, U2 ProMicro

Commit message: Left pcb should be done
Connections:
- net col0: now also U2.13 (10/PB6); no longer U2.20 (A3/PF4)
- net col1: now also U2.14 (16/PB2); no longer U2.19 (A2/PF5)
- net col2: now also U2.15 (14/PB3); no longer U2.18 (A1/PF6)
- net col3: now also U2.16 (15/PB1); no longer U2.17 (A0/PF7)
- net col4: now also U2.17 (A0/PF7); no longer U2.16 (15/PB1)
- net col5: now also U2.18 (A1/PF6); no longer U2.15 (14/PB3)
- net col6: now also U2.19 (A2/PF5); no longer U2.14 (16/PB2)
- net col7: now also U2.20 (A3/PF4); no longer U2.13 (10/PB6)
Changed lines of the file:
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@@
     (effects (font (size 1.27 1.27)) (justify left bottom))
   )
-  (label "col7" (at 91.44 60.96 0)
+  (label "col0" (at 91.44 60.96 0)
     (effects (font (size 1.27 1.27)) (justify left bottom))
   )
-  (label "col2" (at 91.44 48.26 0)
+  (label "col5" (at 91.44 48.26 0)
     (effects (font (size 1.27 1.27)) (justify left bottom))
   )
@@
     (effects (font (size 1.27 1.27)) (justify left bottom))
   )
-  (label "col4" (at 91.44 53.34 0)
+  (label "col3" (at 91.44 53.34 0)
     (effects (font (size 1.27 1.27)) (justify left bottom))
   )
@@
     (effects (font (size 1.27 1.27)) (justify right bottom))
   )
-  (label "col5" (at 91.44 55.88 0)
+  (label "col2" (at 91.44 55.88 0)
     (effects (font (size 1.27 1.27)) (justify left bottom))
   )
-  (label "col1" (at 91.44 45.72 0)
+  (label "col6" (at 91.44 45.72 0)
     (effects (font (size 1.27 1.27)) (justify left bottom))
   )
@@
     (effects (font (size 1.27 1.27)) (justify right bottom))
   )
-  (label "col6" (at 91.44 58.42 0)
+  (label "col1" (at 91.44 58.42 0)
     (effects (font (size 1.27 1.27)) (justify left bottom))
   )
@@
     (effects (font (size 1.27 1.27)) (justify left bottom))
   )
-  (label "col0" (at 91.44 43.18 0)
+  (label "col7" (at 91.44 43.18 0)
     (effects (font (size 1.27 1.27)) (justify left bottom))
   )
@@
     (effects (font (size 1.27 1.27)) (justify left bottom))
   )
-  (label "col3" (at 91.44 50.8 0)
+  (label "col4" (at 91.44 50.8 0)
     (effects (font (size 1.27 1.27)) (justify left bottom))
   )

Commit message: Starting on right pcb
Parts:
- U2: value ProMicro -> ProMicro USBC; footprint keebio:ArduinoProMicro -> keebio:ArduinoProMicro-USBC-Alibaba; symbol keebio:ProMicro -> keebio:ProMicro_usbc_alibaba
Changed lines of the file:
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@@
     (pin "4")
   )
-  (symbol (lib_id "keebio:ProMicro") (at 73.66 46.99 0) (unit 1)
+  (symbol (lib_id "keebio:ProMicro_usbc_alibaba") (at 73.66 46.99 0) (unit 1)
     (in_bom yes) (on_board yes)
     (property "Reference" "U2" (id 0) (at 73.66 25.7302 0)
       (effects (font (size 1.524 1.524)))
     )
-    (property "Value" "ProMicro" (id 1) (at 73.66 28.4226 0)
+    (property "Value" "ProMicro USBC" (id 1) (at 73.66 28.4226 0)
       (effects (font (size 1.524 1.524)))
     )
-    (property "Footprint" "keebio:ArduinoProMicro" (id 2) (at 100.33 110.49 90)
+    (property "Footprint" "keebio:ArduinoProMicro-USBC-Alibaba" (id 2) (at 100.33 110.49 90)
       (effects (font (size 1.524 1.524)) hide)
     )
@@
     )
     (path "/00000000-0000-0000-0000-00005eac825b"
-      (reference "U2") (unit 1) (value "ProMicro") (footprint "keebio:ArduinoProMicro")
-    )
-  )
+      (reference "U2") (unit 1) (value "ProMicro USBC") (footprint "keebio:ArduinoProMicro-USBC-Alibaba")
+    )
+  )
